Commit message: Updated Realsense launch files

File: ros/jetsoncar_description/urdf/jetsoncar.xacro (robot description, xacro)
@@ -221,5 +221,7 @@
         </link>
         <xacro:fixed_offset_joint_rpy parent="realsense_d435_mount_center" child="realsense_t265_mount_center" offset="0 0 0.030" rpy="0 0 0" />
-        <link name="realsense_t265_link">
+        <xacro:fixed_offset_joint_rpy parent="realsense_t265_mount_center" child="realsense_t265_link_" offset="0.00595 0.0091 0" rpy="0 0 0" />
+        <!-- realsense_t265_pose_frame to realsense_t265_link is published by Realsense node -->
+        <link name="realsense_t265_link_">
             <visual>
                     <material name="lightgrey"/>
@@ -230,5 +232,4 @@
             </visual>
         </link>
-        <xacro:fixed_offset_joint_rpy parent="realsense_t265_mount_center" child="realsense_t265_link" offset="0.00595 0.0091 0" rpy="0 0 0" />
     </xacro:if>
 </robot>

Commit message: Added Hokuyo model and update sensor launch files and RVIZ

File: ros/jetsoncar_description/urdf/jetsoncar.xacro (robot description, xacro)
@@ -28,6 +28,6 @@
             <visual>
                 <material name="grey"/>
-                <origin xyz="0.0136 -0.015 0.012" rpy="-${pi/2} 0 -${pi/2}" />
-                <!--<xacro:imu_geometry/>-->
+                <!--<origin xyz="0.0136 -0.015 0.012" rpy="-${pi/2} 0 -${pi/2}" />
+                <xacro:imu_geometry/>-->
                 <geometry>
                     <mesh filename="package://jetsoncar_description/models/spatial.dae" scale="1.0 1.0 1.0"/>
@@ -168,10 +168,17 @@
 		<xacro:fixed_offset_joint parent="base_link" child="lidar_mount" offset="0 0 ${baseplate_thickness}"/>-->
 		<link name="lidar">
-			<visual>
+			<!--<visual>
 				<material name="red"/>
 				<xacro:lidar_geometry/>
-			</visual>
-		</link>
-		<xacro:fixed_offset_joint_rpy parent="base_link" child="lidar" offset="0 0 ${baseplate_thickness+lidar_height/2}" rpy="0 0 ${pi}"/>
+			</visual>-->
+            <visual>
+                <material name="lightgrey"/>
+                <geometry>
+                    <mesh filename="package://jetsoncar_description/models/hokuyo.stl" scale="0.001 0.001 0.001"/>
+                </geometry>
+                <origin rpy="${pi/2} 0 0" xyz="-${lidar_width/2} ${lidar_length/2} -${lidar_scanline_height}"/>
+            </visual>
+		</link>
+		<xacro:fixed_offset_joint_rpy parent="base_link" child="lidar" offset="0 0 ${baseplate_thickness+lidar_scanline_height}" rpy="0 0 ${pi}"/>
 	</xacro:if>
 	<xacro:if value="${enable_range_sensors}">

File: ros/jetsoncar_description/urdf/parameters.xacro (robot description, xacro)
@@ -56,4 +56,5 @@
 	<xacro:property name="lidar_height" value="0.05" />
 	<xacro:property name="lidar_weight" value="0.200" />
+    <xacro:property name="lidar_scanline_height" value="0.057" />
 	<xacro:property name="lidar_mount_diameter" value="0.08" />
 	<xacro:property name="lidar_mount_height" value="0.13" />
